File: pcb_gps_poncho.sch (KiCad schematic (older format))
At the start: 5 parts, among them P1 CONN_5, P2 CONN_4

Commit message: Cambio de chip gps y modelo de poncho
Parts:
- removed H1, H2: PCB_HOLE, Poncho_Modelos:Led_Hole, symbol PCB_HOLE
- added U1?: SE868-A, symbol SE868-A
- added unit 1 of XA1
- XA1: footprint Poncho_Esqueleto:Conn_Poncho_Izquierdo -> (none)
Connections:
- net labels added: +3.3V, +5V
- wire segments 22 -> 31
- no-connect marks 18 -> 31
Other:
- note removed: "Agujeros para visualización de LEDs"
- moved on the sheet: P1, P2, XA1B, XA1K
